File: Cub_Wolf_Badge_Circuit.sch (KiCad schematic (older format))
At the start: 12 parts, among them Q1 2N3904, Q2 2N3904, SW1 SW_SPDT

Commit message: Updated trace placement on switch, updated resistor values.
Parts:
- R1, R4: value 1k -> 220
- R2, R3: value 5k -> 10k
Changed lines of the file:
@@
 P 3425 2775
 F 0 "R1" H 3495 2821 50  0000 L CNN
-F 1 "1k" H 3495 2730 50  0000 L CNN
+F 1 "220" H 3495 2730 50  0000 L CNN
 F 2 "Resistors_THT:R_Axial_DIN0207_L6.3mm_D2.5mm_P10.16mm_Horizontal" V 3355 2775 50  0001 C CNN
 F 3 "~" H 3425 2775 50  0001 C CNN
@@
 P 4900 2775
 F 0 "R4" H 4970 2821 50  0000 L CNN
-F 1 "1k" H 4970 2730 50  0000 L CNN
+F 1 "220" H 4970 2730 50  0000 L CNN
 F 2 "Resistors_THT:R_Axial_DIN0207_L6.3mm_D2.5mm_P10.16mm_Horizontal" V 4830 2775 50  0001 C CNN
 F 3 "~" H 4900 2775 50  0001 C CNN
@@
 P 4025 2825
 F 0 "R2" H 4095 2871 50  0000 L CNN
-F 1 "5k" H 4095 2780 50  0000 L CNN
+F 1 "10k" H 4095 2780 50  0000 L CNN
 F 2 "Resistors_THT:R_Axial_DIN0207_L6.3mm_D2.5mm_P10.16mm_Horizontal" V 3955 2825 50  0001 C CNN
 F 3 "~" H 4025 2825 50  0001 C CNN
@@
 P 4300 2825
 F 0 "R3" H 4370 2871 50  0000 L CNN
-F 1 "5k" H 4370 2780 50  0000 L CNN
+F 1 "10k" H 4370 2780 50  0000 L CNN
 F 2 "Resistors_THT:R_Axial_DIN0207_L6.3mm_D2.5mm_P10.16mm_Horizontal" V 4230 2825 50  0001 C CNN
 F 3 "~" H 4300 2825 50  0001 C CNN
